File: Ultimate macro thing/Ultimate macro thing.sch (KiCad schematic (older format))
At the start: 71 parts, among them J1 Conn_02x03_Odd_Even, J2 Conn_01x04, SW1 SW_Push, SW2 SW_Push, SW3 Rotary_Encoder, U1 ATmega328P-PU, Y1 16Mhz

Commit message: wiring in process
Parts:
- C1: footprint (none) -> Capacitor_THT:CP_Radial_D4.0mm_P1.50mm
- C2, C3: footprint (none) -> Capacitor_THT:C_Disc_D4.3mm_W1.9mm_P5.00mm
- C4, C5: footprint (none) -> Capacitor_THT:C_Disc_D3.0mm_W1.6mm_P2.50mm
- D1, D2: footprint (none) -> Diode_THT:D_DO-35_SOD27_P7.62mm_Horizontal
- D5, D6: footprint (none) -> LED_THT:LED_D3.0mm_Clear
- F1: footprint (none) -> Capacitor_THT:C_Disc_D5.0mm_W2.5mm_P5.00mm
- J1: footprint (none) -> Connector_PinHeader_2.54mm:PinHeader_2x03_P2.54mm_Vertical
- J2: footprint (none) -> Connector_PinHeader_2.54mm:PinHeader_1x04_P2.54mm_Vertical
- MX1, MX10, MX11, MX12, MX13, MX14, MX15, MX2, MX3, MX4, MX6, MX7, MX8, MX9: footprint Bases github:MX-1U-NoLED -> ! MX bases:MXOnly-1U-NoLED
- MX5: footprint (none) -> ! MX bases:MXOnly-1U-NoLED
- R1, R2, R3, R4, R5, R6: footprint (none) -> Resistor_THT:R_Axial_DIN0204_L3.6mm_D1.6mm_P5.08mm_Horizontal
- R7, R8: value I2C -> 10k; footprint (none) -> Resistor_THT:R_Axial_DIN0204_L3.6mm_D1.6mm_P5.08mm_Horizontal
- SW1, SW2: footprint (none) -> Button_Switch_THT:SW_PUSH_6mm
- SW3: footprint (none) -> Rotary_Encoder:RotaryEncoder_Alps_EC11E_Vertical_H20mm
- USB1: footprint (none) -> !random-keyboard-parts:Molex-0548190519
- Y1: footprint (none) -> Crystal:Crystal_HC49-4H_Vertical
Connections:
- net COL1: now also MX5.1 (COL)
